File: board/stm32f7.sch (EAGLE design)
At the start: 22 parts, among them IC1 LM2937, U1 STM32F722XX, X1 MINI-USB-32005-201

Commit message: board
Parts:
- added ADC: (no value), con-lsta:FE10-1
- added C14: 100n, resistor:C-EUC0805
- added D1, D2: (no value), adafruit:DIODE_SOD-123FL
- added IC2: FT232RL, ftdichip:FT232RL
- added LED1: (no value), my_parts:LEDCHIPLED_1206
- added R3: 4k7, resistor:R-EU_M0805
- added SV1: (no value), con-lsta:FE06-2
- added X2: MINI-USB-32005-201, con-cypressindustries:MINI-USB-32005-201
Connections:
- new net ADC0: ADC.1, U1A.PA0
- new net ADC1: ADC.2, U1A.PA1
- new net ADC2: ADC.3, U1A.PA2
- new net ADC3: ADC.4, U1A.PA3
- new net ADC4: ADC.5, U1A.PA4
- new net ADC5: ADC.6, U1A.PA5
- new net ADC6: ADC.7, U1A.PA6
- new net ADC7: ADC.8, U1A.PA7
- new net ADC8: ADC.9, U1A.PB0
- new net ADC9: ADC.10, U1A.PB1
- new net KEY: S2.3
- new net LED: R3.2
- new net N$10: D2.A, X2.1
- new net N$15: SV1.7
- new net N$16: SV1.9
- new net N$17: SV1.11
- new net N$18: SV1.12
- new net N$19: SV1.10
- new net N$20: SV1.8
- new net N$5: LED1.A, R3.1
- new net N$6: C14.1, IC2.3V3OUT, IC2.VCCIO
- new net N$7: D1.A, X1.1
- new net N$8: IC2.USBDM, X2.2
- new net N$9: IC2.USBDP, X2.3
- new net TIM1_CH1: SV1.2, U1A.PE9
- new net TIM1_CH1N: SV1.1, U1A.PE8
- new net TIM1_CH2: SV1.4, U1A.PE11
- new net TIM1_CH2N: SV1.3, U1A.PE10
- new net TIM1_CH3: SV1.6, U1A.PE13
- new net TIM1_CH3N: SV1.5, U1A.PE12
- new net TIM1_CH4: U1A.PE14
- new net TIM2_CH3: U1A.PB10
- new net TIM2_CH4: U1A.PB11
- new net USART1_RX: IC2.TXD, U1B.PA10
- new net USART1_TX: IC2.RXD, U1B.PA9
- new net USBDM: U1B.PA_11, X1.2
- new net USBDP: U1B.PA12, X1.3
- net +5V: now also D1.C, D2.C, IC2.VCC
- net GND: now also C14.2, IC2.GND, IC2.GND@1, IC2.GND@2, IC2.GND@A, IC2.TEST, LED1.C, S1.1, S2.1, X1.5, X2.5
- net RESET: now also S1.3
Other:
- moved on the sheet: BOOT, C1, C10, C11, C12, C13, C2, C3, C4, C5, C6, C7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

Commit message: common
Parts:
- added C15: 10uF, resistor:C-EUC0805
- added C16: 100n, resistor:C-EUC0805
- added C17: 22uF, resistor:CPOL-EU153CLV-0505
- added LED2: (no value), my_parts:LEDCHIPLED_1206
- added R4, R5, R6: 4k7, resistor:R-EU_M0805
- renumbered S1 to RESET, S2 to KEY, SV1 to GPIO
Connections:
- removed net N$15: GPIO.7
- removed net N$16: GPIO.9
- removed net N$17: GPIO.11
- removed net N$18: GPIO.12
- removed net N$19: GPIO.10
- removed net N$20: GPIO.8
- new net N$11: LED2.A, R6.1
- new net SCL: GPIO.7, R5.1, U1B.PC7
- new net SDA: GPIO.8, R4.1, U1B.PC8
- net +3V3: now also C16.1, GPIO.9, R4.2, R5.2, R6.2
- net +5V: now also C15.1, C17.+, GPIO.11
- net GND: now also C15.2, C16.2, C17.-, GPIO.10, GPIO.12, LED2.C
- net KEY: now also U1B.PC9
- net LED: now also U1B.PA8
Other:
- moved on the sheet: D1, X1

Commit message: common
Parts:
- removed ADC: (no value), con-lsta:FE10-1
- removed GPIO: (no value), con-lsta:FE06-2
- removed R4, R5: 4k7, resistor:R-EU_M0805
- added U2: ARDUINOR3-BPLACE, adafruit:ARDUINOR3-BPLACE
Connections:
- new net N$14: U2.D2
- new net N$15: U2.D3
- new net N$16: U2.D4
- new net N$17: U2.D5
- new net N$18: U2.D6
- new net N$19: U2.D7
- new net N$20: U2.D8
- new net N$21: U2.D9
- new net N$22: U2.D10
- new net N$23: U2.D11
- new net N$24: U2.D12
- new net N$25: U2.D13
- net +3V3: now also U2.3V; no longer GPIO.9, R4.2, R5.2
- net +5V: now also U2.5V; no longer GPIO.11
- net ADC0: now also U2.A0; no longer ADC.1
- net ADC1: now also U2.A1; no longer ADC.2
- net ADC2: now also U2.A2; no longer ADC.3
- net ADC3: now also U2.A3; no longer ADC.4
- net ADC4: now also U2.A4/SDA; no longer ADC.5
- net ADC5: now also U2.A5/SCL; no longer ADC.6
- net ADC6: no longer ADC.7
- net ADC7: no longer ADC.8
- net ADC8: no longer ADC.9
- net ADC9: no longer ADC.10
- net GND: now also U2.GND, U2.GND1, U2.GND2; no longer GPIO.10, GPIO.12
- net SCL: no longer GPIO.7, R5.1
- net SDA: no longer GPIO.8, R4.1
- net TIM1_CH1: no longer GPIO.2
- net TIM1_CH1N: no longer GPIO.1
- net TIM1_CH2: no longer GPIO.4
- net TIM1_CH2N: no longer GPIO.3
- net TIM1_CH3: no longer GPIO.6
- net TIM1_CH3N: no longer GPIO.5
- net USART1_RX: now also U2.D0
- net USART1_TX: now also U2.D1

Commit message: board
Parts:
- removed C14: 100n, resistor:C-EUC0805
- removed C15: 10uF, resistor:C-EUC0805
- removed C17: 22uF, resistor:CPOL-EU153CLV-0505
- removed D1, D2: (no value), adafruit:DIODE_SOD-123FL
- removed IC1: LM2937, linear:LM2937
- removed IC2: FT232RL, ftdichip:FT232RL
- removed U2: ARDUINOR3-BPLACE, adafruit:ARDUINOR3-BPLACE
- removed X2: MINI-USB-32005-201, con-cypressindustries:MINI-USB-32005-201
- added U$1: MIC5504-3.3Y, my_parts:MIC5504-3.3Y
Connections:
- removed net N$10: D2.A, X2.1
- removed net N$14: U2.D2
- removed net N$15: U2.D3
- removed net N$16: U2.D4
- removed net N$17: U2.D5
- removed net N$18: U2.D6
- removed net N$19: U2.D7
- removed net N$20: U2.D8
- removed net N$21: U2.D9
- removed net N$22: U2.D10
- removed net N$23: U2.D11
- removed net N$24: U2.D12
- removed net N$25: U2.D13
- removed net N$6: C14.1, IC2.3V3OUT, IC2.VCCIO
- removed net N$7: D1.A, X1.1
- removed net N$8: IC2.USBDM, X2.2
- removed net N$9: IC2.USBDP, X2.3
- net +3V3: now also U$1.VOUT; no longer IC1.VO, U2.3V
- net +5V: now also U$1.EN, U$1.VIN, X1.1; no longer C15.1, C17.+, D1.C, D2.C, IC1.VI, IC2.VCC, U2.5V
- net ADC0: no longer U2.A0
- net ADC1: no longer U2.A1
- net ADC2: no longer U2.A2
- net ADC3: no longer U2.A3
- net ADC4: no longer U2.A4/SDA
- net ADC5: no longer U2.A5/SCL
- net GND: now also U$1.GND; no longer C14.2, C15.2, C17.-, IC1.GND, IC2.GND, IC2.GND@1, IC2.GND@2, IC2.GND@A, IC2.TEST, U2.GND, U2.GND1, U2.GND2, X2.5
- net USART1_RX: no longer IC2.TXD, U2.D0
- net USART1_TX: no longer IC2.RXD, U2.D1
Other:
- moved on the sheet: BOOT, C12, C13, C16, C3, C6, C7, C8, C9, KEY, LED1, LED2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

Commit message: board
Parts:
- removed KEY: DTSM-6, switch-tact:DTSM-6
- added C14: 10n, resistor:C-EUC0805
- added C15: 100n, resistor:C-EUC0805
- added GPIO: (no value), con-lstb:MA04-2
- added I2C, USART: (no value), con-lstb:MA04-1
- added R4, R5: 4k7, resistor:R-EU_M0805
- added U$2: ST_L3GD20H, main:ST_L3GD20H
- Q1: value (none) -> 8MHz
Connections:
- new net N$6: C14.1, U$2.CAP
- net +3V3: now also C15.1, GPIO.1, I2C.3, R4.2, R5.2, U$2.CS, U$2.VDD, U$2.VDD_IO, USART.4
- net ADC0: now also GPIO.4
- net ADC1: now also GPIO.3
- net ADC2: now also GPIO.6
- net ADC3: now also GPIO.5
- net ADC4: now also GPIO.8
- net ADC5: now also GPIO.7
- net GND: now also C14.2, C15.2, GPIO.2, I2C.4, U$2.DEN, U$2.GND, U$2.RES1, U$2.RES2, U$2.RES3, U$2.RES4, U$2.SDO, USART.1; no longer KEY.1
- net KEY: no longer KEY.3
- net SCL: now also I2C.2, R5.1, U$2.SCL/SPC, U1B.PB7; no longer U1B.PC7
- net SDA: now also I2C.1, R4.1, U$2.SDA/SDI, U1B.PB6; no longer U1B.PC8
- net USART1_RX: now also USART.3
- net USART1_TX: now also USART.2
