File: board/stm32f7.brd (EAGLE design)
At the start: 49.7 x 49.8 mm, 31 parts, among them IC1 LM2937, IC2 FT232RL, U1 STM32F722XX, X1 MINI-USB-32005-201, X2 MINI-USB-32005-201

Commit message: common
Parts:
- added C15: 10uF, resistor:C0805
- added C16: 100n, resistor:C0805
- added C17: 22uF, resistor:153CLV-0505
- added LED2: (no value), my_parts:CHIPLED_1206
- added R4, R5, R6: 4k7, resistor:M0805
- moved C14 18.6 mm to (14.3, 38.1), turned to 270 degrees
- moved R3 6.82 mm to (37.2, 33.5), turned to 270 degrees
- moved R2 4.07 mm to (7.32, 14.3)
- moved IC2 1.85 mm to (15.5, 31.7), turned to 180 degrees
- moved D1 1.64 mm to (12.2, 47.5), turned to 180 degrees
- moved LED1 1.36 mm to (36.6, 36.9)
- moved BOOT 1.29 mm to (3.66, 17.4), turned to 0 degrees
- moved C7 0.43 mm to (34.4, 21.6)
- renumbered S1 to RESET, S2 to KEY, SV1 to GPIO
Connections:
- removed net N$15: GPIO.7
- removed net N$16: GPIO.9
- removed net N$17: GPIO.11
- removed net N$18: GPIO.12
- removed net N$19: GPIO.10
- removed net N$20: GPIO.8
- new net N$11: LED2.A, R6.1
- new net SCL: GPIO.7, R5.1, U1.64
- new net SDA: GPIO.8, R4.1, U1.65
- net +3V3: now also C16.1, GPIO.9, R4.2, R5.2, R6.2
- net +5V: now also C15.1, C17.+, GPIO.11
- net GND: now also C15.2, C16.2, C17.-, GPIO.10, GPIO.12, LED2.C
- net KEY: now also U1.66
- net LED: now also U1.67
Routing:
- net GND: track 109.4 -> 267.0 mm, vias 6 -> 33
- net +3V3: track 66.3 -> 159.0 mm, vias 6 -> 7
- net +5V: track 5.24 -> 97.2 mm, vias 0 -> 3
- net USBDM: track 0.00 -> 39.6 mm
- net USBDP: track 0.00 -> 38.0 mm
- net BOOT: track 2.51 -> 37.9 mm
- net USART1_TX: track 0.00 -> 28.7 mm, vias 0 -> 2
- net TIM1_CH1N: track 0.00 -> 26.9 mm, vias 0 -> 1
- net TIM1_CH1: track 0.00 -> 25.4 mm, vias 0 -> 1
- net TIM1_CH2N: track 0.00 -> 25.1 mm, vias 0 -> 1
- net USART1_RX: track 0.00 -> 25.1 mm, vias 0 -> 2
- net TIM1_CH2: track 0.00 -> 24.8 mm, vias 0 -> 1
- net N$6: track 0.00 -> 23.4 mm
- net TIM1_CH3N: track 0.00 -> 21.7 mm, vias 0 -> 2
- net TIM1_CH3: track 0.00 -> 20.7 mm
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- added copper zone on layer 1, net GND
- added copper zone on layer 16, net GND
Other:
- board text added: "3V3"
- board text added: "5V"
- board text added: "ADC0"
- board text added: "ADC9"
- board text added: "GND"
- board text added: "SCL"

Commit message: common
Parts:
- removed ADC: (no value), con-lsta:FE10
- removed GPIO: (no value), con-lsta:FE06-2
- removed R4, R5: 4k7, resistor:M0805
- added U2: ARDUINOR3-BPLACE, adafruit:ARDUINOR3-BPLACE
- moved KEY 25.6 mm to (64.3, 27.4)
- moved R2 18.6 mm to (25.9, 15.2), turned to 0 degrees
- moved C3 14.1 mm to (26.0, 6.20)
- moved C5 14.0 mm to (46.0, 31.7)
- moved C7 14.0 mm to (48.5, 21.0)
- moved C8 14.0 mm to (40.5, 28.7)
- moved C9 14.0 mm to (36.6, 18.0)
- moved R1 14.0 mm to (30.2, 5.59)
- moved U1 14.0 mm to (42.8, 19.6)
- moved C1 14.0 mm to (26.0, 8.59)
- moved C2 14.0 mm to (25.8, 12.8)
- moved C6 14.0 mm to (44.8, 14.6)
- moved Q1 14.0 mm to (30.1, 10.7)
- moved C4 14.0 mm to (54.6, 16.8)
- moved R3 5.33 mm to (41.8, 36.3), turned to 0 degrees
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Connections:
- new net N$14: U2.D2
- new net N$15: U2.D3
- new net N$16: U2.D4
- new net N$17: U2.D5
- new net N$18: U2.D6
- new net N$19: U2.D7
- new net N$20: U2.D8
- new net N$21: U2.D9
- new net N$22: U2.D10
- new net N$23: U2.D11
- new net N$24: U2.D12
- new net N$25: U2.D13
- new net VIN: U2.VIN
- net +3V3: now also U2.3V; no longer GPIO.9, R4.2, R5.2
- net +5V: now also U2.5V; no longer GPIO.11
- net ADC0: now also U2.A0; no longer ADC.1
- net ADC1: now also U2.A1; no longer ADC.2
- net ADC2: now also U2.A2; no longer ADC.3
- net ADC3: now also U2.A3; no longer ADC.4
- net ADC4: now also U2.A4; no longer ADC.5
- net ADC5: now also U2.A5; no longer ADC.6
- net ADC6: no longer ADC.7
- net ADC7: no longer ADC.8
- net ADC8: no longer ADC.9
- net ADC9: no longer ADC.10
- net GND: now also U2.GND, U2.GND1, U2.GND2; no longer GPIO.10, GPIO.12
- net SCL: no longer GPIO.7, R5.1
- net SDA: no longer GPIO.8, R4.1
- net TIM1_CH1: no longer GPIO.2
- net TIM1_CH1N: no longer GPIO.1
- net TIM1_CH2: no longer GPIO.4
- net TIM1_CH2N: no longer GPIO.3
- net TIM1_CH3: no longer GPIO.6
- net TIM1_CH3N: no longer GPIO.5
- net USART1_RX: now also U2.D0
- net USART1_TX: now also U2.D1
Routing:
- net GND: track 267.0 -> 321.9 mm, vias 33 -> 23
- net USART1_RX: track 25.1 -> 76.0 mm
- net USART1_TX: track 28.7 -> 72.5 mm
- net TIM1_CH1N: track 26.9 -> 0.00 mm, vias 1 -> 0
- net TIM1_CH1: track 25.4 -> 0.00 mm, vias 1 -> 0
- net TIM1_CH2N: track 25.1 -> 0.00 mm, vias 1 -> 0
- net TIM1_CH2: track 24.8 -> 0.00 mm, vias 1 -> 0
- net TIM1_CH3N: track 21.7 -> 0.00 mm, vias 2 -> 0
- net TIM1_CH3: track 20.7 -> 0.00 mm
- net KEY: track 19.8 -> 0.00 mm
- net ADC3: track 8.31 -> 24.0 mm
- net SDA: track 15.4 -> 0.00 mm
- net ADC9: track 15.0 -> 0.00 mm
- net USBDP: track 38.0 -> 52.8 mm
- net USBDM: track 39.6 -> 54.2 mm
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- removed copper zone on layer 1, net GND
- removed copper zone on layer 16, net GND
Other:
- board outline removed
- board text removed: "3V3"
- board text removed: "5V"
- board text removed: "ADC0"
- board text removed: "ADC9"
- board text removed: "GND"
- board text removed: "SCL"

Commit message: board
Parts:
- removed C14: 100n, resistor:C0805
- removed C15: 10uF, resistor:C0805
- removed C17: 22uF, resistor:153CLV-0505
- removed D1, D2: (no value), adafruit:SOD-123FL
- removed IC1: LM2937, linear:TO263-3
- removed IC2: FT232RL, ftdichip:SSOP28
- removed U2: ARDUINOR3-BPLACE, adafruit:ARDUINOR3-BPLACE
- removed X2: MINI-USB-32005-201, con-cypressindustries:32005-201
- added U$1: MIC5504-3.3Y, my_parts:SOT23-5
- moved RESET 60.4 mm to (65.2, 14.5), turned to 0 degrees
- moved C10 43.7 mm to (65.8, 57.1)
- moved C11 43.7 mm to (63.0, 57.1)
- moved C12 43.7 mm to (65.8, 52.8)
- moved C13 43.7 mm to (63.0, 52.8)
- moved C16 43.7 mm to (68.2, 44.0)
- moved LED2 43.7 mm to (71.0, 48.6)
- moved R3 43.7 mm to (83.8, 48.3)
- moved R6 43.7 mm to (66.4, 49.5)
- moved X1 43.7 mm to (47.2, 55.0)
- moved LED1 43.7 mm to (78.9, 48.3)
- moved C8 18.7 mm to (22.3, 25.0)
- moved C1 18.7 mm to (7.67, 4.93)
- moved C2 18.7 mm to (7.52, 9.09)
- moved C3 18.7 mm to (7.72, 2.54)
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Connections:
- removed net N$10: D2.A, X2.1
- removed net N$14: U2.D2
- removed net N$15: U2.D3
- removed net N$16: U2.D4
- removed net N$17: U2.D5
- removed net N$18: U2.D6
- removed net N$19: U2.D7
- removed net N$20: U2.D8
- removed net N$21: U2.D9
- removed net N$22: U2.D10
- removed net N$23: U2.D11
- removed net N$24: U2.D12
- removed net N$25: U2.D13
- removed net N$6: C14.1, IC2.17, IC2.4
- removed net N$7: D1.A, X1.1
- removed net N$8: IC2.16, X2.2
- removed net N$9: IC2.15, X2.3
- removed net VIN: U2.VIN
- net +3V3: now also U$1.P$5; no longer IC1.3, U2.3V
- net +5V: now also U$1.P$1, U$1.P$3, X1.1; no longer C15.1, C17.+, D1.C, D2.C, IC1.1, IC2.20, U2.5V
- net ADC0: no longer U2.A0
- net ADC1: no longer U2.A1
- net ADC2: no longer U2.A2
- net ADC3: no longer U2.A3
- net ADC4: no longer U2.A4
- net ADC5: no longer U2.A5
- net GND: now also U$1.P$2; no longer C14.2, C15.2, C17.-, IC1.2, IC2.18, IC2.21, IC2.25, IC2.26, IC2.7, U2.GND, U2.GND1, U2.GND2, X2.5
- net USART1_RX: no longer IC2.1, U2.D0
- net USART1_TX: no longer IC2.5, U2.D1
Routing:
- net GND: track 321.9 -> 190.2 mm, vias 23 -> 16
- net +5V: track 104.5 -> 23.0 mm, vias 3 -> 1
- net USART1_RX: track 76.0 -> 5.64 mm, vias 2 -> 1
- net USART1_TX: track 72.5 -> 8.14 mm, vias 2 -> 1
- net +3V3: track 162.3 -> 106.3 mm, vias 8 -> 7
- net RESET: track 45.3 -> 19.2 mm
- net N$6: track 23.4 -> 0.00 mm
- net BOOT: track 39.8 -> 19.2 mm
- net USBDM: track 54.2 -> 40.3 mm
- net USBDP: track 52.8 -> 38.9 mm
- net LED: track 21.6 -> 12.8 mm
- net N$10: track 7.50 -> 0.00 mm
- net N$8: track 6.27 -> 0.00 mm
- net N$9: track 5.04 -> 0.00 mm
- net N$7: track 4.71 -> 0.00 mm
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Other:
- board outline added: 38 x 37.7 mm

Commit message: board
Parts:
- removed KEY: DTSM-6, switch-tact:DTSM-6
- added C14: 10n, resistor:C0805
- added C15: 100n, resistor:C0805
- added GPIO: (no value), con-lstb:MA04-2
- added I2C, USART: (no value), con-lstb:MA04-1
- added R4, R5: 4k7, resistor:M0805
- added U$2: ST_L3GD20H, main:ST_LGA16L
- Q1: value (none) -> 8MHz
- moved RESET 60.2 mm to (5.52, 22.6)
- moved C10 55.2 mm to (15.2, 35.0)
- moved U$1 54.8 mm to (18.9, 35.1)
- moved C11 54.8 mm to (12.9, 34.9)
- moved C16 51.1 mm to (19.4, 28.8)
- moved R3 50.7 mm to (35.4, 33.3), turned to 180 degrees
- moved X1 48.0 mm to (5.12, 31.8)
- moved C12 47.1 mm to (22.1, 35.2), turned to 270 degrees
- moved LED1 46.0 mm to (34.7, 35.6)
- moved LED2 43.8 mm to (29.1, 35.5), turned to 90 degrees
- moved C13 42.5 mm to (24.3, 35.2), turned to 270 degrees
- moved R6 39.8 mm to (30.1, 33.2)
- moved BOOT 1.45 mm to (3.17, 3.10), turned to 180 degrees
Connections:
- new net N$6: C14.1, U$2.P$14
- net +3V3: now also C15.1, GPIO.1, I2C.3, R4.2, R5.2, U$2.P$1, U$2.P$16, U$2.P$5, USART.4
- net ADC0: now also GPIO.4
- net ADC1: now also GPIO.3
- net ADC2: now also GPIO.6
- net ADC3: now also GPIO.5
- net ADC4: now also GPIO.8
- net ADC5: now also GPIO.7
- net GND: now also C14.2, C15.2, GPIO.2, I2C.4, U$2.P$10, U$2.P$11, U$2.P$12, U$2.P$13, U$2.P$15, U$2.P$4, U$2.P$8, U$2.P$9, USART.1; no longer KEY.1
- net KEY: no longer KEY.3
- net SCL: now also I2C.2, R5.1, U$2.P$2, U1.93; no longer U1.64
- net SDA: now also I2C.1, R4.1, U$2.P$3, U1.92; no longer U1.65
- net USART1_RX: now also USART.3
- net USART1_TX: now also USART.2
Routing:
- net +3V3: track 106.3 -> 194.9 mm, vias 7 -> 13
- net GND: track 190.2 -> 227.7 mm, vias 16 -> 21
- net SCL: track 0.00 -> 36.0 mm, vias 0 -> 1
- net RESET: track 19.2 -> 49.7 mm, vias 0 -> 2
- net SDA: track 0.00 -> 21.2 mm
- net USBDP: track 38.9 -> 28.2 mm
- net ADC4: track 19.5 -> 8.84 mm
- net USBDM: track 40.3 -> 29.7 mm
- net ADC5: track 21.8 -> 11.8 mm
- net BOOT: track 19.2 -> 27.6 mm
- net USART1_RX: track 5.64 -> 13.3 mm, vias 1 -> 2
- net +5V: track 23.0 -> 15.5 mm, vias 1 -> 0
- net ADC2: track 22.2 -> 15.8 mm
- net ADC3: track 23.1 -> 18.3 mm
- net N$6: track 0.00 -> 2.87 mm
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- added copper zone on layer 1, net GND
- added copper zone on layer 16, net GND

Commit message: ir cam
Routing:
- net GND: track 227.7 -> 228.4 mm
- net +3V3: vias 13 -> 12
Changed lines of the file:
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@@
 <setting verticaltext="up"/>
 </settings>
-<grid distance="10" unitdist="mil" unit="mil" style="lines" multiple="1" display="no" altdistance="0.025" altunitdist="inch" altunit="inch"/>
+<grid distance="8" unitdist="mil" unit="mil" style="lines" multiple="1" display="yes" altdistance="0.025" altunitdist="inch" altunit="inch"/>
 <layers>
 <layer number="1" name="Top" color="4" fill="1" visible="yes" active="yes"/>
@@
 <wire x1="31.3944" y1="14.6304" x2="32.3088" y2="14.6304" width="0.3048" layer="1"/>
 <wire x1="32.3088" y1="14.6304" x2="32.6136" y2="14.9352" width="0.3048" layer="1"/>
-<wire x1="33.296459375" y1="14.9352" x2="33.843025" y2="14.388634375" width="0.3048" layer="1"/>
 <wire x1="23.4696" y1="10.0584" x2="22.2504" y2="11.2776" width="0.3048" layer="16"/>
 <via x="22.2504" y="11.2776" extent="1-16" drill="0.6"/>
@@
 <wire x1="22.2504" y1="11.2776" x2="22.2504" y2="10.668" width="0.3048" layer="1"/>
 <wire x1="22.2504" y1="10.668" x2="21.6408" y2="10.0584" width="0.3048" layer="1"/>
-<wire x1="21.6408" y1="10.0584" x2="21.6408" y2="8.86771875" width="0.3048" layer="1"/>
 <wire x1="21.6408" y1="8.86771875" x2="21.14494375" y2="8.3718625" width="0.3048" layer="1"/>
 <wire x1="30.48" y1="15.5448" x2="30.48" y2="16.1544" width="0.6096" layer="16"/>
@@
 <contactref element="C16" pad="2"/>
 <contactref element="LED2" pad="C"/>
-<wire x1="32.6136" y1="14.9352" x2="33.296459375" y2="14.9352" width="0.3048" layer="1"/>
 <wire x1="7.9248" y1="11.2776" x2="7.6962" y2="11.5062" width="0.6096" layer="16"/>
 <via x="6.4008" y="12.8016" extent="1-16" drill="0.6"/>
@@
 <vertex x="-10.16" y="-18.034"/>
 </polygon>
+<wire x1="21.6408" y1="8.86771875" x2="21.66931875" y2="8.86771875" width="0.254" layer="1"/>
+<wire x1="21.66931875" y1="8.86771875" x2="21.9456" y2="9.144" width="0.254" layer="1"/>
+<wire x1="21.9456" y1="9.144" x2="21.9456" y2="9.3472" width="0.254" layer="1"/>
+<wire x1="21.9456" y1="9.3472" x2="21.7424" y2="9.5504" width="0.254" layer="1"/>
+<wire x1="21.7424" y1="9.5504" x2="21.7424" y2="9.7536" width="0.254" layer="1"/>
+<wire x1="21.7424" y1="9.7536" x2="21.5392" y2="9.9568" width="0.254" layer="1"/>
+<wire x1="21.5392" y1="9.9568" x2="21.6408" y2="10.0584" width="0.254" layer="1"/>
+<wire x1="32.6136" y1="14.9352" x2="32.7152" y2="15.0368" width="0.254" layer="1"/>
+<wire x1="33.843025" y1="14.388634375" x2="33.843025" y2="14.416975" width="0.254" layer="1"/>
+<wire x1="33.843025" y1="14.416975" x2="33.274" y2="14.986" width="0.254" layer="1"/>
+<wire x1="33.296459375" y1="14.9352" x2="33.296459375" y2="14.963540625" width="0.254" layer="1"/>
+<wire x1="33.296459375" y1="14.963540625" x2="33.02" y2="15.24" width="0.254" layer="1"/>
+<wire x1="33.02" y1="15.24" x2="32.766" y2="14.986" width="0.254" layer="1"/>
 </signal>
 <signal name="RESET">
@@
 <wire x1="11.988" y1="24.218" x2="13.686" y2="25.916" width="0.3048" layer="1"/>
 <wire x1="15.986" y1="25.116" x2="15.986" y2="23.384" width="0.3048" layer="1"/>
-<wire x1="15.986" y1="23.384" x2="16.002" y2="23.368" width="0.3048" layer="1"/>
-<via x="16.002" y="23.368" extent="1-16" drill="0.6"/>
 <wire x1="15.51" y1="23.384" x2="14.478" y2="22.352" width="0.3048" layer="16"/>
 <wire x1="14.478" y1="22.352" x2="11.684" y2="22.352" width="0.3048" layer="16"/>
@@
 <wire x1="10.668" y1="23.876" x2="11.342" y2="23.876" width="0.3048" layer="1"/>
 <wire x1="11.342" y1="23.876" x2="11.684" y2="24.218" width="0.3048" layer="1"/>
-<wire x1="16.002" y1="23.368" x2="18.034" y2="25.4" width="0.3048" layer="16"/>
 <via x="18.034" y="25.4" extent="1-16" drill="0.6"/>
 <wire x1="18.034" y1="25.4" x2="18.796" y2="25.4" width="0.3048" layer="1"/>
@@
 <via x="15.986" y="23.384" extent="1-16" drill="0.6"/>
 <wire x1="15.986" y1="23.384" x2="15.51" y2="23.384" width="0.3048" layer="16"/>
+<wire x1="18.034" y1="25.4" x2="18.002" y2="25.4" width="0.3048" layer="16"/>
+<wire x1="18.002" y1="25.4" x2="15.986" y2="23.384" width="0.3048" layer="16"/>
 </signal>
 <signal name="BOOT">
