File: ascender_board/ascender_board.brd (EAGLE design)
At the start: 94 x 80 mm, 89 parts, among them Q1 8MHz, U1 STM32F722XX, U2 LM5107MA, U3 LM5107MA, U4 LM5107MA, U5 LM5107MA, U6 LM5107MA, U7 LM5107MA, X1 MINI-USB-32005-201

Commit message: board
Parts:
- moved U5 76.4 mm to (80.9, 5.81), turned to 0 degrees
- moved C34 72.3 mm to (72.9, 3.81), turned to 0 degrees
- moved C32 72.1 mm to (75.9, 5.81), turned to 0 degrees
- moved U7 70.0 mm to (80.9, 11.5), turned to 0 degrees
- moved C26 67.7 mm to (69.9, 5.81), turned to 0 degrees
- moved R14 67.6 mm to (75.9, 9.81), turned to 0 degrees
- moved C28 67.4 mm to (72.9, 7.81), turned to 0 degrees
- moved C30 65.8 mm to (66.9, 5.81), turned to 0 degrees
- moved R13 65.3 mm to (75.9, 11.8), turned to 0 degrees
- moved C33 65.1 mm to (81.0, 10.1), turned to 0 degrees
- moved C31 64.9 mm to (62.9, 4.81), turned to 0 degrees
- moved R16 62.1 mm to (75.9, 14.8), turned to 0 degrees
- moved C27 60.8 mm to (71.9, 12.8), turned to 0 degrees
- moved R15 59.6 mm to (68.9, 11.8), turned to 0 degrees
- moved C25 59.1 mm to (58.9, 7.81), turned to 270 degrees
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Routing:
- net VCC: track 0.00 -> 81.3 mm
- net GND: track 226.9 -> 304.9 mm
- net N$25: track 0.00 -> 60.5 mm, vias 0 -> 3
- net N$19: track 0.00 -> 59.9 mm, vias 0 -> 3
- net N$16: track 0.00 -> 59.1 mm, vias 0 -> 3
- net N$17: track 0.00 -> 2.81 mm
- net N$7: track 0.00 -> 2.76 mm
- net N$20: track 0.00 -> 2.61 mm
- net N$8: track 0.00 -> 2.49 mm
- net N$23: track 0.00 -> 2.43 mm
- net N$12: track 0.00 -> 2.38 mm

Commit message: board
Parts:
- added U$22, U$23, U$24, U$25: SI7210, my_parts:SOT23-5
- moved R13 65.6 mm to (13.0, 30.4), turned to 180 degrees
- moved R15 62.3 mm to (13.1, 39.5), turned to 180 degrees
- moved R16 59.7 mm to (21.6, 39.5), turned to 180 degrees
- moved R17 58.9 mm to (12.9, 21.2), turned to 180 degrees
- moved R14 57.8 mm to (21.9, 30.3), turned to 180 degrees
- moved U5 50.6 mm to (33.7, 24.0), turned to 90 degrees
- moved C32 45.0 mm to (33.0, 19.6), turned to 180 degrees
- moved C23 43.7 mm to (33.7, 47.7), turned to 180 degrees
- moved C28 43.5 mm to (38.7, 34.6), turned to 270 degrees
- moved LED1 42.8 mm to (50.3, 54.2)
- moved C33 42.0 mm to (39.2, 13.7), turned to 270 degrees
- moved C26 41.7 mm to (35.0, 28.5), turned to 180 degrees
- moved C25 39.2 mm to (41.1, 42.7), turned to 90 degrees
- moved U7 38.3 mm to (42.7, 13.8), turned to 90 degrees
- moved R3 38.1 mm to (52.7, 54.5), turned to 270 degrees
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Connections:
- removed net TIM1_CH1: U1.39
- removed net TIM1_CH1N: U1.38
- removed net TIM1_CH2: U1.41
- removed net TIM1_CH2N: U1.40
- removed net TIM1_CH3: U1.43
- removed net TIM1_CH3N: U1.42
- removed net TIM1_CH4: U1.44
- removed net TIM2_CH3: U1.46
- removed net TIM2_CH4: U1.47
- new net SCL_ENC: U$22.P$3, U$23.P$3, U$24.P$3, U$25.P$3, U1.1
- new net SDA_0_ENC: U$22.P$1, U1.2
- new net SDA_1_ENC: U$23.P$1, U1.3
- new net SDA_2_ENC: U$24.P$1, U1.4
- new net SDA_3_ENC: U$25.P$1, U1.5
- net +3V3: now also U$22.P$4, U$23.P$4, U$24.P$4, U$25.P$4
- net GND: now also U$22.P$2, U$23.P$2, U$24.P$2, U$25.P$2
- net UH_LEFT: now also U1.39
- net UH_RIGHT: now also U1.44
- net UL_LEFT: now also U1.38
- net UL_RIGHT: now also U1.45
- net VH_LEFT: now also U1.41
- net VH_RIGHT: now also U1.46
- net VL_LEFT: now also U1.40
- net VL_RIGHT: now also U1.37
- net WH_LEFT: now also U1.43
- net WH_RIGHT: now also U1.47
- net WL_LEFT: now also U1.42
- net WL_RIGHT: now also U1.36
Routing:
- net N$37: track 0.00 -> 54.9 mm, vias 0 -> 3
- net N$43: track 0.00 -> 53.8 mm, vias 0 -> 3
- net N$31: track 0.00 -> 53.4 mm, vias 0 -> 3
- net GND: track 304.9 -> 327.8 mm
- net VCC: track 81.3 -> 103.5 mm
- net N$38: track 0.00 -> 2.89 mm
- net N$29: track 0.00 -> 2.54 mm
- net N$35: track 0.00 -> 2.50 mm
- net N$26: track 0.00 -> 2.49 mm
- net N$32: track 0.00 -> 2.42 mm

Commit message: board
Parts:
- added X2: 52745-1890, con-molex:52745-1890
- moved U$25 9.81 mm to (40.5, 69.4), turned to 180 degrees
- moved U$23 8.00 mm to (40.8, 10.7)
- moved U$24 6.26 mm to (18.6, 69.3)
- moved U7 6.14 mm to (45.8, 19.1)
- moved U$22 6.01 mm to (18.9, 10.7)
- moved C33 5.38 mm to (34.1, 15.5)
- moved C34 3.62 mm to (39.1, 14.7), turned to 180 degrees

Commit message: board
Parts:
- removed R10, R11, R12, R13, R14, R15, R16, R17, R18, R7, R8, R9: 0, resistor:M0805
- moved C22 5.33 mm to (44.1, 53.4)
- moved C21 4.57 mm to (41.0, 53.4)
- moved C19 3.83 mm to (42.4, 65.1), turned to 270 degrees
- moved C18 3.69 mm to (39.9, 65.2), turned to 270 degrees
- moved U4 3.20 mm to (34.0, 45.8), turned to 0 degrees
- moved C25 3.12 mm to (43.9, 44.1), turned to 270 degrees
- moved C24 2.45 mm to (40.5, 43.8), turned to 270 degrees
- moved U3 2.17 mm to (34.1, 54.1), turned to 0 degrees
- moved C23 1.98 mm to (32.9, 49.5), turned to 0 degrees
- moved U2 0.76 mm to (33.7, 63.0)
- moved C20 0.61 mm to (33.3, 58.1), turned to 0 degrees
- moved C17 0.53 mm to (32.6, 67.3), turned to 0 degrees
Connections:
- removed net N$12: R8.1, U$4.4
- removed net N$13: R9.2, U3.5
- removed net N$17: R10.1, U$7.4
- removed net N$21: R11.2, U4.5
- removed net N$23: R12.1, U$10.4
- removed net N$26: R13.1, U$14.4
- removed net N$29: R14.1, U$13.4
- removed net N$33: R15.2, U6.5
- removed net N$35: R16.1, U$16.4
- removed net N$39: R17.2, U7.5
- removed net N$41: R18.1, U$19.4
- removed net N$8: R7.1, U$5.4
- net N$10: now also U$4.4; no longer R8.2
- net N$14: now also U$7.4; no longer R10.2
- net N$20: now also U4.5; no longer R11.1
- net N$22: now also U$10.4; no longer R12.2
- net N$27: now also U$14.4; no longer R13.2
- net N$28: now also U$13.4; no longer R14.2
- net N$32: now also U6.5; no longer R15.1
- net N$34: now also U$16.4; no longer R16.2
- net N$38: now also U7.5; no longer R17.1
- net N$40: now also U$19.4; no longer R18.2
- net N$7: now also U3.5; no longer R9.1
- net N$9: now also U$5.4; no longer R7.2
Routing:
- net N$17: track 2.81 -> 0.00 mm
- net N$7: track 2.76 -> 0.00 mm
- net N$20: track 2.61 -> 0.00 mm
- net N$38: track 2.89 -> 0.31 mm
- net N$29: track 2.54 -> 0.00 mm
- net N$35: track 2.50 -> 0.00 mm
- net N$8: track 2.49 -> 0.00 mm
- net N$26: track 2.49 -> 0.00 mm
- net N$23: track 2.43 -> 0.00 mm
- net N$32: track 2.42 -> 0.00 mm
- net N$12: track 2.38 -> 0.00 mm
