File: ascender_board_dc/ascender_board.sch (EAGLE design)
At the start: 92 parts, among them Q1 8MHz, U1 STM32F722XX, U2 LM5107MA, U3 LM5107MA, U4 LM5107MA, U5 LM5107MA, U6 LM5107MA, U7 LM5107MA, X1 MINI-USB-32005-201

Commit message: common
Parts:
- removed C24, C27, C30, C33: 100n, resistor:C-EUC0805
- removed C25, C28, C31, C34: 10uF, resistor:C-EUC0805
- removed C26, C29, C32: 1uF, resistor:C-EUC0805
- removed GPIO: (no value), con-lstb:MA04-2
- removed I2C: (no value), con-lstb:MA04-1
- removed R10, R11, R12, R13, R14, R15, R16, R17, R18, R8, R9: 0, resistor:R-EU_M0805
- removed U$11, U$13, U$14, U$16, U$17, U$19, U$20, U$4, U$5, U$7, U$8: IRFH7004, my_parts:IRFH7004
- removed U$12, U$15, U$18, U$21, U$6, U$9: BLDC_MOTOR_PIN, my_parts:BLDC_MOTOR_PIN
- removed U$22, U$23, U$24, U$25: SI7210, my_parts:SI7210
- removed U2, U3, U4, U5, U6, U7: LM5107MA, my_parts:LM5107MA
- added BAT: LiPol, jumper:JP1E
- added IC1: LM2937, my_parts:LM2937
- added IC2: MC33932, freescale:MC33932
- added X2, X3: 52745-1890, con-molex:52745-1890
- C17, C23: value 1uF -> 100n
- C19: value 10uF -> 100n
- C20: value 1uF -> (none); device resistor:C-EUC0805 -> resistor:CPOL-EU153CLV-0505
- C21: value 100n -> (none); device resistor:C-EUC0805 -> resistor:CPOL-EU153CLV-0505
- C22: value 10uF -> (none); device resistor:C-EUC0805 -> resistor:CPOL-EU153CLV-0505
- R7: value 0 -> 4k7
- U$1: value MIC5504-3.3Y -> POLOLU_GEAR_MOTORPOLO; device my_parts:MIC5504-3.3Y -> my_parts:POLOLU_GEAR_MOTORPOLO
- U$10: value IRFH7004 -> POLOLU_GEAR_MOTORPOLO; device my_parts:IRFH7004 -> my_parts:POLOLU_GEAR_MOTORPOLO
Connections:
- removed net N$13: R9.2, U3.LO
- removed net N$15: C17.2, U2.HB
- removed net N$16: C17.1, U$4.S, U$5.D, U$6.P$1, U2.HS
- removed net N$17: R10.1, U$7.G
- removed net N$18: C20.2, U3.HB
- removed net N$19: C20.1, U$7.S, U$8.D, U$9.P$1, U3.HS
- removed net N$20: R11.1, U$11.G
- removed net N$21: R11.2, U4.LO
- removed net N$22: R12.2, U4.HO
- removed net N$23: R12.1, U$10.G
- removed net N$24: C23.2, U4.HB
- removed net N$25: C23.1, U$10.S, U$11.D, U$12.P$1, U4.HS
- removed net N$26: R13.1, U$14.G
- removed net N$27: R13.2, U5.LO
- removed net N$28: R14.2, U5.HO
- removed net N$29: R14.1, U$13.G
- removed net N$30: C26.2, U5.HB
- removed net N$31: C26.1, U$13.S, U$14.D, U$15.P$1, U5.HS
- removed net N$32: R15.1, U$17.G
- removed net N$33: R15.2, U6.LO
- removed net N$34: R16.2, U6.HO
- removed net N$35: R16.1, U$16.G
- removed net N$36: C29.2, U6.HB
- removed net N$37: C29.1, U$16.S, U$17.D, U$18.P$1, U6.HS
- removed net N$38: R17.1, U$20.G
- removed net N$39: R17.2, U7.LO
- removed net N$40: R18.2, U7.HO
- removed net N$41: R18.1, U$19.G
- removed net N$42: C32.2, U7.HB
- removed net N$43: C32.1, U$19.S, U$20.D, U$21.P$1, U7.HS
- removed net SCL_ENC: U$22.SCL, U$23.SCL, U$24.SCL, U$25.SCL
- removed net SDA_0_ENC: U$22.SDA
- removed net SDA_1_ENC: U$23.SDA
- removed net SDA_2_ENC: U$24.SDA
- removed net SDA_3_ENC: U$25.SDA
- removed net UH_LEFT: U1A.PE9, U2.HI
- removed net UH_RIGHT: U1A.PE14, U5.HI
- removed net UL_LEFT: U1A.PE8, U2.LI
- removed net UL_RIGHT: U1A.PE15, U5.LI
- removed net VH_LEFT: U1A.PE11, U3.HI
- removed net VH_RIGHT: U1A.PB10, U6.HI
- removed net VL_LEFT: U1A.PE10, U3.LI
- removed net VL_RIGHT: U1A.PE7, U6.LI
- removed net WH_LEFT: U1A.PE13, U4.HI
- removed net WH_RIGHT: U1A.PB11, U7.HI
- removed net WL_LEFT: U1A.PE12, U4.LI
- removed net WL_RIGHT: U1A.PB2, U7.LI
- new net ENC_A_LEFT: U$10.A, U1A.PE3
- new net ENC_A_RIGHT: U$1.A, U1A.PE5
- new net ENC_B_LEFT: U$10.B, U1A.PE4
- new net ENC_B_RIGHT: U$1.B, U1A.PE6
- new net FRONT_GPIO: X2-3.S
- new net MOTOR_ENABLE: IC2.EN/!D2, IC2.EN/!D4, R7.2, U1A.PE14
- new net PWM_A_LEFT: IC2.IN1, U1A.PE12
- new net PWM_A_RIGHT: IC2.IN3, U1A.PE10
- new net PWM_B_LEFT: IC2.IN2, U1A.PE13
- new net PWM_B_RIGHT: IC2.IN4, U1A.PE11
- net +3V3: now also C22.+, IC1.VO, U$1.VCC, U$10.VCC, X2-18.S; no longer GPIO.1, I2C.3, U$1.VOUT, U$22.VCC, U$23.VCC, U$24.VCC, U$25.VCC
- net +5V: no longer C10.1, C11.1, U$1.EN, U$1.VIN
- net ADC0: no longer GPIO.4
- net ADC1: no longer GPIO.3
- net ADC2: no longer GPIO.6
- net ADC3: no longer GPIO.5
- net ADC4: no longer GPIO.8
- net ADC5: no longer GPIO.7
- net GND: now also BAT.1, C20.-, C21.-, C22.-, C23.2, IC1.GND, IC2.D1, IC2.D3, IC2.EH@1, IC2.EH@2, IC2.EH@3, IC2.PGNDA, IC2.PGNDA@1, IC2.PGNDA@2, IC2.PGNDA@3, IC2.PGNDB, IC2.PGNDB@1, IC2.PGNDB@2, IC2.PGNDB@3, R7.1, U$10.GND, X2-17.S; no longer C18.2, C21.2, C22.2, C24.2, C25.2, C27.2, C28.2, C30.2, C31.2, C33.2, C34.2, GPIO.2, I2C.4, U$11.S, U$14.S, U$17.S, U$20.S, U$22.GND, U$23.GND, U$24.GND, U$25.GND, U$5.S, U$8.S, U2.VSS, U3.VSS, U4.VSS, U5.VSS, U6.VSS, U7.VSS
- net N$10: now also IC2.OUT3, IC2.OUT3@1, IC2.OUT3@2, U$1.P$1; no longer R8.2, U2.HO
- net N$12: now also C17.2, IC2.CCPA; no longer R8.1, U$4.G
- net N$14: now also C18.1, IC2.CCPB; no longer R10.2, U3.HO
- net N$7: now also IC2.OUT1, IC2.OUT1@1, IC2.OUT1@2, U$10.P$1; no longer R9.1, U$8.G
- net N$8: now also IC2.OUT2, IC2.OUT2@1, IC2.OUT2@2, U$10.P$2; no longer R7.1, U$5.G
- net N$9: now also IC2.OUT4, IC2.OUT4@1, IC2.OUT4@2, U$1.P$2; no longer R7.2, U2.LO
- net SCL: now also X2-1.S; no longer I2C.2
- net SDA: now also X2-2.S; no longer I2C.1
- net VCC: now also BAT.2, C10.1, C11.1, C17.1, C18.2, C20.+, C21.+, C23.1, IC1.VI, IC2.VPWRA, IC2.VPWRA@1, IC2.VPWRA@2, IC2.VPWRA@3, IC2.VPWRA@4, IC2.VPWRB, IC2.VPWRB@1, IC2.VPWRB@2, IC2.VPWRB@3, IC2.VPWRB@4; no longer C18.1, C21.1, C22.1, C24.1, C25.1, C27.1, C28.1, C30.1, C31.1, C33.1, C34.1, U$10.D, U$13.D, U$16.D, U$19.D, U$4.D, U$7.D, U2.VDD, U3.VDD, U4.VDD, U5.VDD, U6.VDD, U7.VDD
Other:
- moved on the sheet: C12, C13, C17, C18, C19, C23, R7

Commit message: board
Parts:
- removed X1: MINI-USB-32005-201, con-cypressindustries:MINI-USB-32005-201
- added C24: (no value), resistor:CPOL-EU153CLV-0505
- added C25: 10uF, resistor:C-EUC0805
- added C26: 100n, resistor:C-EUC0805
- added CAMERA: (no value), con-lsta:FE06-1
- added D1: (no value), diode:DIODE-DO-214AC
- added LED3, LED4, LED5, LED6, LED7: (no value), my_parts:LEDCHIPLED_1206
- added Q2, Q3, Q4: BSS123, transistor-small-signal:BSS123
- added R10, R11, R12, R18, R8, R9: 4k7, resistor:R-EU_M0805
- added R13, R14, R15, R16, R19: 330, resistor:R-EU_M0805
- added R17: 22, resistor:R-EU_M0805
- added RUN: DTSM-6, switch-tact:DTSM-6
- added U$11: SFH3710, my_parts:SFH3710
- added U$12: KPA3010, my_parts:KPA3010
- added U$13: KPA3010_EM, my_parts:KPA3010_EM
- added U$3, U$4, U$5, U$6, U$7, U$8: FIDUCIAL, adafruit:FIDUCIAL
- added U$9: TSOP4830, tsop:TSOP4830
- added U2: I2C EEPROM, SparkFun-IC-Memory:EEPROM-I2CEIAJ
- added X4: MINI-USB-SCHIELD-32005-201, con-cypressindustries:MINI-USB-SCHIELD-32005-201
Connections:
- removed net +5V: X1.1
- new net ADC10: U1A.PB0, X2-14.S
- new net ADC11: CAMERA.3, U1A.PB1
- new net ADC1_S: R18.1, U$11.C, X3-14.S
- new net CAM_CLK: CAMERA.5, U1A.PE9
- new net CAM_SI: CAMERA.6, U1A.PE8
- new net FRONT_SCL: U1A.PC0, X2-1.S
- new net FRONT_SDA: U1A.PC1, X2-2.S
- new net IR_A: Q2.D, X2-15.S
- new net IR_A_CONTROLL: Q2.G, R10.2, U1A.PB2
- new net IR_A_S: R19.1, X3-4.S
- new net IR_B: Q3.D, X2-16.S
- new net IR_B_CONTROLL: Q3.G, R11.2, U1A.PE7
- new net IR_REMOTE: U$9.OUT, U1A.PE2
- new net LED_BACK: Q4.G, R12.2, U1B.PD13
- new net N$13: IC2.FBA, R8.2
- new net N$15: IC2.FBB, R9.1
- new net N$16: LED3.C, LED4.C, LED5.C, LED6.C, Q4.D
- new net N$17: LED3.A, R13.1
- new net N$18: D1.A, X4G$1.1
- new net N$19: LED4.A, R14.1
- new net N$20: C25.1, R17.1, U$9.V+
- new net N$21: LED5.A, R15.1
- new net N$23: LED6.A, R16.1
- new net N$24: LED7.C, R19.2
- new net NC: CAMERA.4
- net +3V3: now also C24.+, C26.1, CAMERA.1, LED7.A, R13.2, R14.2, R15.2, R16.2, R17.2, R18.2, U2.VCC, U2.WP, X2-17.S, X3-2.S; no longer X2-18.S
- net ADC0: now also X2-4.S
- net ADC1: now also X2-5.S
- net ADC2: now also X2-6.S
- net ADC3: now also X2-7.S
- net ADC4: now also X2-8.S
- net ADC5: now also X2-9.S
- net ADC6: now also X2-10.S
- net ADC7: now also X2-11.S
- net ADC8: now also U1A.PC4, X2-12.S; no longer U1A.PB0
- net ADC9: now also U1A.PC5, X2-13.S; no longer U1A.PB1
- net ENC_A_LEFT: now also U1B.PC6; no longer U1A.PE3
- net ENC_A_RIGHT: now also U1B.PB4; no longer U1A.PE5
- net ENC_B_LEFT: now also U1B.PC7; no longer U1A.PE4
- net ENC_B_RIGHT: now also U1B.PB5; no longer U1A.PE6
- net FRONT_GPIO: now also U1A.PC2
- net GND: now also C24.-, C25.2, C26.2, CAMERA.2, Q2.S, Q3.S, Q4.S, R10.1, R11.1, R12.1, R8.1, R9.2, RUN.1, U$11.E, U$9.GND, U2.A0, U2.A1, U2.A2, U2.VSS, X2-18.S, X3-1.S, X4G$1.5, X4S.S1, X4S.S2, X4S.S3, X4S.S4; no longer X1.5, X2-17.S
- net KEY: now also RUN.3, U1A.PE3; no longer U1B.PC9
- net MOTOR_ENABLE: now also U1B.PD0; no longer U1A.PE14
- net SCL: now also U1B.PD2, U2.SCL; no longer U1B.PB7, X2-1.S
- net SDA: now also U1B.PD1, U2.SDA; no longer U1B.PB6, X2-2.S
- net USBDM: now also X4G$1.2; no longer X1.2
- net USBDP: now also X4G$1.3; no longer X1.3
- net VCC: now also D1.C
Other:
- moved on the sheet: C1, C14, C15, C16, C2, C3, C4, C5, C6, C7, C8, C9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

Commit message: board
Parts:
- added H1, H2, H3, H4: MOUNT-HOLE3.0, holes:MOUNT-HOLE3.0
- added LED10, LED11, LED12, LED13, LED14, LED8, LED9: (no value), my_parts:LEDCHIPLED_1206
- added R20, R22, R24, R26, R28, R30, R32, R34, R36, R38: 4k7, resistor:R-EU_M0805
- added R21, R23, R25, R27, R29, R31, R33: 330, resistor:R-EU_M0805
- added R35, R37, R39: 22, resistor:R-EU_M0805
- added U$14, U$15, U$16, U$17, U$18, U$19, U$20: SFH3710, my_parts:SFH3710
- added U$29, U$31: KPA3010, my_parts:KPA3010
- added U$30, U$32: KPA3010_EM, my_parts:KPA3010_EM
Connections:
- new net ADC2_S: R20.1, U$14.C, X3-13.S
- new net ADC3_S: R22.1, U$15.C, X3-12.S
- new net ADC4_S: R24.1, U$16.C, X3-11.S
- new net ADC6_S: R26.1, U$17.C, X3-9.S
- new net ADC7_S: R28.1, U$18.C, X3-8.S
- new net ADC8_S: R30.1, U$19.C, X3-7.S
- new net ADC9_S: R32.1, U$20.C, X3-6.S
- new net IR_B_S: U$13.C, U$30.C, U$32.C, X3-3.S
- new net IR_FRONT_S: R36.1, U$29.P$1, X3-10.S
- new net IR_LEFT_S: R38.1, U$31.P$1, X3-5.S
- new net IR_RIGHT_S: R34.1, U$12.P$1, X3-15.S
- new net N$22: LED8.C, R21.2
- new net N$25: LED9.C, R23.2
- new net N$26: LED10.C, R25.2
- new net N$27: LED11.C, R27.2
- new net N$28: LED12.C, R29.2
- new net N$29: LED13.C, R31.2
- new net N$30: LED14.C, R33.2
- new net N$31: R37.1, U$30.A
- new net N$32: R35.1, U$13.A
- new net N$33: R39.1, U$32.A
- net +3V3: now also LED10.A, LED11.A, LED12.A, LED13.A, LED14.A, LED8.A, LED9.A, R20.2, R22.2, R24.2, R26.2, R28.2, R30.2, R32.2, R34.2, R35.2, R36.2, R37.2, R38.2, R39.2
- net GND: now also U$12.P$2, U$14.E, U$15.E, U$16.E, U$17.E, U$18.E, U$19.E, U$20.E, U$29.P$2, U$31.P$2
- net IR_A_CONTROLL: now also U1A.PE7; no longer U1A.PB2
- net IR_A_S: now also R21.1, R23.1, R25.1, R27.1, R29.1, R31.1, R33.1
- net IR_B_CONTROLL: now also U1A.PB2; no longer U1A.PE7
Other:
- moved on the sheet: LED7, R18, R19, U$13
