File: ascender_board_dc/ascender_board.brd (EAGLE design)
At the start: 94 x 80 mm, 82 parts, among them Q1 8MHz, U1 STM32F722XX, U2 LM5107MA, U3 LM5107MA, U4 LM5107MA, U5 LM5107MA, U6 LM5107MA, U7 LM5107MA, X1 MINI-USB-32005-201, X2 52745-1890

Commit message: common
Parts:
- removed C24, C27, C30, C33: 100n, resistor:C0805
- removed C25, C28, C31, C34: 10uF, resistor:C0805
- removed C26, C29, C32: 1uF, resistor:C0805
- removed GPIO: (no value), con-lstb:MA04-2
- removed I2C: (no value), con-lstb:MA04-1
- removed U$11, U$13, U$14, U$16, U$17, U$19, U$20, U$4, U$5, U$7, U$8: IRFH7004, my_parts:PQFN5X6
- removed U$12, U$15, U$18, U$21, U$6, U$9: BLDC_MOTOR_PIN, my_parts:BLDC_MOTOR_PIN
- removed U$22, U$23, U$24, U$25: SI7210, my_parts:SOT23-5
- removed U$3: (no value), mechanical:BLDC_MOTOR_HOLDER
- removed U2, U3, U4, U5, U6, U7: LM5107MA, my_parts:SOIC127P620X175-8N
- added BAT: LiPol, jumper:JP1
- added IC1: LM2937, my_parts:TO263-3
- added IC2: MC33932, freescale:HSOP44
- added R7: 4k7, resistor:M0805
- added X3: 52745-1890, con-molex:52745-1890
- C17, C23: value 1uF -> 100n
- C19: value 10uF -> 100n
- C20: value 1uF -> (none); device resistor:C0805 -> resistor:153CLV-0505
- C21: value 100n -> (none); device resistor:C0805 -> resistor:153CLV-0505
- C22: value 10uF -> (none); device resistor:C0805 -> resistor:153CLV-0505
- U$1: value MIC5504-3.3Y -> POLOLU_GEAR_MOTORPOLO; device my_parts:SOT23-5 -> my_parts:POLOLU_GEAR_MOTOR
- U$10: value IRFH7004 -> POLOLU_GEAR_MOTORPOLO; device my_parts:PQFN5X6 -> my_parts:POLOLU_GEAR_MOTOR
- moved C18 63.5 mm to (56.9, 5.84), flipped to the top, turned to 270 degrees
- moved USART 54.3 mm to (10.0, 34.1), turned to 90 degrees
- moved C19 53.9 mm to (35.1, 12.2), flipped to the top, turned to 270 degrees
- moved X1 53.3 mm to (5.25, 45.5), turned to 0 degrees
- moved C20 52.5 mm to (35.1, 5.33), flipped to the top, turned to 270 degrees
- moved C17 51.8 mm to (37.1, 16.3), flipped to the top, turned to 270 degrees
- moved LED2 51.2 mm to (2.43, 30.5)
- moved LED1 50.9 mm to (2.55, 36.7)
- moved C12 50.9 mm to (6.69, 15.8), flipped to the bottom, turned to 270 degrees
- moved R6 50.7 mm to (5.45, 31.0)
- moved R3 50.4 mm to (5.42, 37.0)
- moved C13 49.8 mm to (9.18, 15.9), flipped to the bottom, turned to 270 degrees
- moved C11 48.8 mm to (6.79, 11.4), flipped to the bottom, turned to 90 degrees
- moved C10 47.7 mm to (9.08, 11.5), flipped to the bottom, turned to 90 degrees
- moved C23 45.4 mm to (29.0, 2.54), flipped to the top, turned to 90 degrees
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Connections:
- removed net N$13: U3.5
- removed net N$15: C17.2, U2.8
- removed net N$16: C17.1, U$4.1, U$4.2, U$4.3, U$5.5, U$5.6, U$5.7, U$5.8, U$6.P$1, U2.6
- removed net N$17: U$7.4
- removed net N$18: C20.2, U3.8
- removed net N$19: C20.1, U$7.1, U$7.2, U$7.3, U$8.5, U$8.6, U$8.7, U$8.8, U$9.P$1, U3.6
- removed net N$20: U$11.4, U4.5
- removed net N$22: U$10.4, U4.7
- removed net N$24: C23.2, U4.8
- removed net N$25: C23.1, U$10.1, U$10.2, U$10.3, U$11.5, U$11.6, U$11.7, U$11.8, U$12.P$1, U4.6
- removed net N$26: U$14.4
- removed net N$27: U5.5
- removed net N$28: U5.7
- removed net N$29: U$13.4
- removed net N$30: C26.2, U5.8
- removed net N$31: C26.1, U$13.1, U$13.2, U$13.3, U$14.5, U$14.6, U$14.7, U$14.8, U$15.P$1, U5.6
- removed net N$32: U$17.4
- removed net N$33: U6.5
- removed net N$34: U6.7
- removed net N$35: U$16.4
- removed net N$36: C29.2, U6.8
- removed net N$37: C29.1, U$16.1, U$16.2, U$16.3, U$17.5, U$17.6, U$17.7, U$17.8, U$18.P$1, U6.6
- removed net N$38: U$20.4, U7.5
- removed net N$40: U$19.4, U7.7
- removed net N$42: C32.2, U7.8
- removed net N$43: C32.1, U$19.1, U$19.2, U$19.3, U$20.5, U$20.6, U$20.7, U$20.8, U$21.P$1, U7.6
- removed net SCL_ENC: U$22.P$3, U$23.P$3, U$24.P$3, U$25.P$3, U1.1
- removed net SDA_0_ENC: U$22.P$1, U1.2
- removed net SDA_1_ENC: U$23.P$1, U1.3
- removed net SDA_2_ENC: U$24.P$1, U1.4
- removed net SDA_3_ENC: U$25.P$1, U1.5
- removed net UH_LEFT: U1.39, U2.2
- removed net UH_RIGHT: U1.44, U5.2
- removed net UL_LEFT: U1.38, U2.3
- removed net UL_RIGHT: U1.45, U5.3
- removed net VH_LEFT: U1.41, U3.2
- removed net VH_RIGHT: U1.46, U6.2
- removed net VL_LEFT: U1.40, U3.3
- removed net VL_RIGHT: U1.37, U6.3
- removed net WH_LEFT: U1.43, U4.2
- removed net WH_RIGHT: U1.47, U7.2
- removed net WL_LEFT: U1.42, U4.3
- removed net WL_RIGHT: U1.36, U7.3
- new net ENC_A_LEFT: U$10.P$4, U1.2
- new net ENC_A_RIGHT: U$1.P$4, U1.4
- new net ENC_B_LEFT: U$10.P$5, U1.3
- new net ENC_B_RIGHT: U$1.P$5, U1.5
- new net FRONT_GPIO: X2.3
- new net MOTOR_ENABLE: IC2.25, IC2.3, R7.2, U1.44
- new net PWM_A_LEFT: IC2.43, U1.42
- new net PWM_A_RIGHT: IC2.21, U1.40
- new net PWM_B_LEFT: IC2.42, U1.43
- new net PWM_B_RIGHT: IC2.20, U1.41
- net +3V3: now also C22.+, IC1.3, U$1.P$3, U$10.P$3, X2.18; no longer GPIO.1, I2C.3, U$1.P$5, U$22.P$4, U$23.P$4, U$24.P$4, U$25.P$4
- net +5V: no longer C10.1, C11.1, U$1.P$1, U$1.P$3
- net ADC0: no longer GPIO.4
- net ADC1: no longer GPIO.3
- net ADC2: no longer GPIO.6
- net ADC3: no longer GPIO.5
- net ADC4: no longer GPIO.8
- net ADC5: no longer GPIO.7
- net GND: now also BAT.1, C20.-, C21.-, C22.-, C23.2, IC1.2, IC2.1, IC2.10, IC2.11, IC2.12, IC2.13, IC2.23, IC2.32, IC2.33, IC2.34, IC2.35, IC2.EH@1, IC2.EH@2, IC2.EH@3, R7.1, U$1.P$6, U$10.P$6, X2.17; no longer C18.2, C21.2, C22.2, C24.2, C25.2, C27.2, C28.2, C30.2, C31.2, C33.2, C34.2, GPIO.2, I2C.4, U$1.P$2, U$11.1, U$11.2, U$11.3, U$14.1, U$14.2, U$14.3, U$17.1, U$17.2, U$17.3, U$20.1, U$20.2, U$20.3, U$22.P$2, U$23.P$2, U$24.P$2, U$25.P$2, U$5.1, U$5.2, U$5.3, U$8.1, U$8.2, U$8.3, U2.4, U3.4, U4.4, U5.4, U6.4, U7.4
- net N$10: now also IC2.29, IC2.30, IC2.31, U$1.P$1; no longer U2.7
- net N$12: now also C17.2, IC2.41; no longer U$4.4
- net N$14: now also C18.1, IC2.19; no longer U3.7
- net N$7: now also IC2.7, IC2.8, IC2.9, U$10.P$1; no longer U$8.4
- net N$8: now also IC2.36, IC2.37, IC2.38, U$10.P$2; no longer U$5.4
- net N$9: now also IC2.14, IC2.15, IC2.16, U$1.P$2; no longer U2.5
- net SCL: now also X2.1; no longer I2C.2
- net SDA: now also X2.2; no longer I2C.1
- net VCC: now also BAT.2, C10.1, C11.1, C17.1, C18.2, C20.+, C21.+, C23.1, IC1.1, IC2.17, IC2.18, IC2.26, IC2.27, IC2.28, IC2.39, IC2.4, IC2.40, IC2.5, IC2.6; no longer C18.1, C21.1, C22.1, C24.1, C25.1, C27.1, C28.1, C30.1, C31.1, C33.1, C34.1, U$10.5, U$10.6, U$10.7, U$10.8, U$13.5, U$13.6, U$13.7, U$13.8, U$16.5, U$16.6, U$16.7, U$16.8, U$19.5, U$19.6, U$19.7, U$19.8, U$4.5, U$4.6, U$4.7, U$4.8, U$7.5, U$7.6, U$7.7, U$7.8, U2.1, U3.1, U4.1, U5.1, U6.1, U7.1
Routing:
- net N$25: track 60.5 -> 0.00 mm, vias 3 -> 0
- net N$19: track 59.9 -> 0.00 mm, vias 3 -> 0
- net N$16: track 59.1 -> 0.00 mm, vias 3 -> 0
- net N$37: track 54.9 -> 0.00 mm, vias 3 -> 0
- net N$43: track 53.8 -> 0.00 mm, vias 3 -> 0
- net N$31: track 53.4 -> 0.00 mm, vias 3 -> 0
- net PWM_A_RIGHT: track 0.00 -> 46.2 mm, vias 0 -> 1
- net VCC: track 103.5 -> 149.1 mm
- net MOTOR_ENABLE: track 0.00 -> 44.5 mm, vias 0 -> 2
- net PWM_B_RIGHT: track 0.00 -> 41.8 mm, vias 0 -> 1
- net GND: track 327.8 -> 359.1 mm, vias 21 -> 17
- net N$9: track 0.00 -> 30.2 mm, vias 0 -> 1
- net USBDM: track 29.7 -> 5.55 mm
- net N$10: track 0.00 -> 24.1 mm, vias 0 -> 1
- net USBDP: track 28.2 -> 4.63 mm
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
Commit message: board
Parts:
- removed X1: MINI-USB-32005-201, con-cypressindustries:32005-201
- added C24: (no value), resistor:153CLV-0505
- added C25: 10uF, resistor:C0805
- added C26: 100n, resistor:C0805
- added CAMERA: (no value), con-lsta:FE06
- added D1: (no value), diode:DO-214AC
- added LED3, LED4, LED5, LED6, LED7: (no value), my_parts:CHIPLED_1206
- added Q2, Q3, Q4: BSS123, transistor-small-signal:SOT23
- added R10, R11, R12, R18, R8, R9: 4k7, resistor:M0805
- added R13, R14, R15, R16, R19: 330, resistor:M0805
- added R17: 22, resistor:M0805
- added RUN: DTSM-6, switch-tact:DTSM-6
- added U$11: SFH3710, my_parts:SFH3710
- added U$12: KPA3010, my_parts:KPA3010
- added U$13: KPA3010_EM, my_parts:KPA3010
- added U$3, U$4, U$5, U$6, U$7, U$8: FIDUCIAL, adafruit:FIDUCIAL_1MM
- added U$9: TSOP4830, tsop:TSOP18XX
- added U2: I2C EEPROM, SparkFun-IC-Memory:SO08-EIAJ
- added X4: MINI-USB-SCHIELD-32005-201, con-cypressindustries:32005-201
- moved RESET 27.9 mm to (88.7, 43.1), turned to 0 degrees
- moved BOOT 22.3 mm to (88.6, 50.6), turned to 90 degrees
- moved R4 6.39 mm to (61.3, 29.6), turned to 0 degrees
- moved X3 3.82 mm to (47.0, 58.4)
- moved R5 3.52 mm to (61.4, 31.9), turned to 0 degrees
- moved R6 3.10 mm to (7.99, 32.7)
- moved LED2 3.09 mm to (5.47, 31.0)
- moved LED1 2.81 mm to (5.35, 36.9)
- moved C15 2.54 mm to (57.8, 27.0)
- moved R3 2.54 mm to (7.46, 38.5)
- moved U$2 2.54 mm to (54.5, 24.0)
- moved X2 2.05 mm to (47.0, 54.9)
- moved C14 1.91 mm to (58.6, 23.7), turned to 180 degrees
- moved USART 1.83 mm to (11.0, 35.6)
- moved C4 1.30 mm to (32.9, 38.5)
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Connections:
- removed net +5V: X1.1
- new net ADC10: U1.34, X2.14
- new net ADC11: CAMERA.3, U1.35
- new net ADC1_S: R18.1, U$11.P$2, X3.14
- new net CAM_CLK: CAMERA.5, U1.39
- new net CAM_SI: CAMERA.6, U1.38
- new net FRONT_SCL: U1.15, X2.1
- new net FRONT_SDA: U1.16, X2.2
- new net IR_A: Q2.3, X2.15
- new net IR_A_CONTROLL: Q2.1, R10.2, U1.36
- new net IR_A_S: R19.1, X3.4
- new net IR_B: Q3.3, X2.16
- new net IR_B_CONTROLL: Q3.1, R11.2, U1.37
- new net IR_REMOTE: U$9.OUT, U1.1
- new net LED_BACK: Q4.1, R12.2, U1.60
- new net N$13: IC2.2, R8.2
- new net N$15: IC2.24, R9.1
- new net N$16: LED3.C, LED4.C, LED5.C, LED6.C, Q4.3
- new net N$17: LED3.A, R13.1
- new net N$18: D1.A, X4.1
- new net N$19: LED4.A, R14.1
- new net N$20: C25.1, R17.1, U$9.VCC
- new net N$21: LED5.A, R15.1
- new net N$23: LED6.A, R16.1
- new net N$24: LED7.C, R19.2
- new net NC: CAMERA.4
- net +3V3: now also C24.+, C26.1, CAMERA.1, LED7.A, R13.2, R14.2, R15.2, R16.2, R17.2, R18.2, U2.7, U2.8, X2.17, X3.2; no longer X2.18
- net ADC0: now also X2.4
- net ADC1: now also X2.5
- net ADC2: now also X2.6
- net ADC3: now also X2.7
- net ADC4: now also X2.8
- net ADC5: now also X2.9
- net ADC6: now also X2.10
- net ADC7: now also X2.11
- net ADC8: now also U1.32, X2.12; no longer U1.34
- net ADC9: now also U1.33, X2.13; no longer U1.35
- net ENC_A_LEFT: now also U1.63; no longer U1.2
- net ENC_A_RIGHT: now also U1.90; no longer U1.4
- net ENC_B_LEFT: now also U1.64; no longer U1.3
- net ENC_B_RIGHT: now also U1.91; no longer U1.5
- net FRONT_GPIO: now also U1.17
- net GND: now also C24.-, C25.2, C26.2, CAMERA.2, Q2.2, Q3.2, Q4.2, R10.1, R11.1, R12.1, R8.1, R9.2, RUN.1, U$11.P$1, U$9.GND, U2.1, U2.2, U2.3, U2.4, X2.18, X3.1, X4.5, X4.M1, X4.M2, X4.M3, X4.M4; no longer X1.5, X2.17
- net KEY: now also RUN.3, U1.2; no longer U1.66
- net MOTOR_ENABLE: now also U1.81; no longer U1.44
- net SCL: now also U1.83, U2.6; no longer U1.93, X2.1
- net SDA: now also U1.82, U2.5; no longer U1.92, X2.2
- net USBDM: now also X4.2; no longer X1.2
- net USBDP: now also X4.3; no longer X1.3
- net VCC: now also D1.C
Routing:
- net GND: track 359.1 -> 659.2 mm, vias 17 -> 48
- net +3V3: track 179.5 -> 470.3 mm, vias 13 -> 22
- net N$16: track 0.00 -> 219.8 mm, vias 0 -> 5
- net IR_REMOTE: track 0.00 -> 58.0 mm, vias 0 -> 2
- net PWM_A_LEFT: track 0.00 -> 42.5 mm, vias 0 -> 2
- net ENC_B_RIGHT: track 0.00 -> 41.8 mm
- net USBDP: track 4.63 -> 46.4 mm
- net N$18: track 0.00 -> 40.6 mm, vias 0 -> 1
- net USBDM: track 5.55 -> 46.0 mm
- net PWM_B_LEFT: track 0.00 -> 39.8 mm, vias 0 -> 2
- net ENC_A_RIGHT: track 0.00 -> 38.6 mm
- net USART1_RX: track 0.00 -> 38.1 mm, vias 0 -> 4
- net KEY: track 0.00 -> 35.7 mm, vias 0 -> 2
- net LED: track 3.85 -> 38.9 mm, vias 1 -> 2
- net PWM_A_RIGHT: track 46.2 -> 80.6 mm, vias 1 -> 2
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- added copper zone on layer 1, net GND
- added copper zone on layer 16, net GND
Other:
- board size 94 x 80 mm -> 94 x 56.6 mm
- board text added: "+"
- board text added: "-"

Commit message: board
Parts:
- added H1, H2, H3, H4: MOUNT-HOLE3.0, holes:3,0
- added LED10, LED11, LED12, LED13, LED14, LED8, LED9: (no value), my_parts:CHIPLED_1206
- added R20, R22, R24, R26, R28, R30, R32, R34, R36, R38: 4k7, resistor:M0805
- added R21, R23, R25, R27, R29, R31, R33: 330, resistor:M0805
- added R35, R37, R39: 22, resistor:M0805
- added U$14, U$15, U$16, U$17, U$18, U$19, U$20: SFH3710, my_parts:SFH3710
- added U$29, U$31: KPA3010, my_parts:KPA3010
- added U$30, U$32: KPA3010_EM, my_parts:KPA3010
- moved U$13 49.6 mm to (43.7, 80.0), turned to 0 degrees
- moved R18 11.6 mm to (83.7, 74.0), turned to 90 degrees
- moved R19 11.4 mm to (80.9, 74.3), turned to 90 degrees
- moved Q2 11.2 mm to (22.4, 52.1), turned to 180 degrees
- moved R10 10.8 mm to (22.4, 55.1), turned to 0 degrees
- moved R1 10.7 mm to (66.2, 43.8), turned to 90 degrees
- moved C24 9.40 mm to (15.0, 52.3)
- moved C3 8.84 mm to (68.5, 43.7), turned to 90 degrees
- moved U$11 5.97 mm to (83.7, 74.3)
- moved LED7 5.97 mm to (80.9, 74.0)
- moved Q3 5.47 mm to (27.7, 53.3), turned to 0 degrees
- moved U$12 3.25 mm to (87.4, 71.5)
- moved R2 3.12 mm to (61.3, 37.0), turned to 270 degrees
- moved R11 2.27 mm to (27.7, 50.3), turned to 180 degrees
- moved C1 1.27 mm to (61.5, 45.4)
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Connections:
- new net ADC2_S: R20.1, U$14.P$2, X3.13
- new net ADC3_S: R22.1, U$15.P$2, X3.12
- new net ADC4_S: R24.1, U$16.P$2, X3.11
- new net ADC6_S: R26.1, U$17.P$2, X3.9
- new net ADC7_S: R28.1, U$18.P$2, X3.8
- new net ADC8_S: R30.1, U$19.P$2, X3.7
- new net ADC9_S: R32.1, U$20.P$2, X3.6
- new net IR_B_S: U$13.P$1_COL, U$30.P$1_COL, U$32.P$1_COL, X3.3
- new net IR_FRONT_S: R36.1, U$29.P$1_COL, X3.10
- new net IR_LEFT_S: R38.1, U$31.P$1_COL, X3.5
- new net IR_RIGHT_S: R34.1, U$12.P$1_COL, X3.15
- new net N$22: LED8.C, R21.2
- new net N$25: LED9.C, R23.2
- new net N$26: LED10.C, R25.2
- new net N$27: LED11.C, R27.2
- new net N$28: LED12.C, R29.2
- new net N$29: LED13.C, R31.2
- new net N$30: LED14.C, R33.2
- new net N$31: R37.1, U$30.P$2_EM, U$30.P$3-NC
- new net N$32: R35.1, U$13.P$2_EM, U$13.P$3-NC
- new net N$33: R39.1, U$32.P$2_EM, U$32.P$3-NC
- net +3V3: now also LED10.A, LED11.A, LED12.A, LED13.A, LED14.A, LED8.A, LED9.A, R20.2, R22.2, R24.2, R26.2, R28.2, R30.2, R32.2, R34.2, R35.2, R36.2, R37.2, R38.2, R39.2
- net GND: now also U$12.P$2_EM, U$12.P$3-NC, U$14.P$1, U$15.P$1, U$16.P$1, U$17.P$1, U$18.P$1, U$19.P$1, U$20.P$1, U$29.P$2_EM, U$29.P$3-NC, U$31.P$2_EM, U$31.P$3-NC
- net IR_A_CONTROLL: now also U1.37; no longer U1.36
- net IR_A_S: now also R21.1, R23.1, R25.1, R27.1, R29.1, R31.1, R33.1
- net IR_B_CONTROLL: now also U1.36; no longer U1.37
Routing:
- net IR_A_S: track 0.00 -> 202.2 mm, vias 0 -> 6
- net GND: track 659.2 -> 828.4 mm, vias 48 -> 66
- net +3V3: track 470.3 -> 632.8 mm, vias 22 -> 33
- net IR_B_S: track 0.00 -> 146.4 mm
- net IR_RIGHT_S: track 0.00 -> 51.6 mm
- net IR_LEFT_S: track 0.00 -> 47.2 mm
- net ADC1_S: track 0.00 -> 46.2 mm, vias 0 -> 1
- net ADC9_S: track 0.00 -> 45.8 mm, vias 0 -> 1
- net ADC8_S: track 0.00 -> 37.2 mm, vias 0 -> 1
- net ADC2_S: track 0.00 -> 36.6 mm, vias 0 -> 1
- net ADC7_S: track 0.00 -> 28.1 mm, vias 0 -> 1
- net ADC3_S: track 0.00 -> 27.7 mm, vias 0 -> 1
- net IR_FRONT_S: track 0.00 -> 21.2 mm
- net ADC6_S: track 0.00 -> 18.3 mm, vias 0 -> 1
- net ADC4_S: track 0.00 -> 17.8 mm, vias 0 -> 1
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Other:
- board size 94 x 56.6 mm -> 94 x 82.8 mm

Commit message: board
Parts:
- added U$21, U$22, U$24: (no value), shapes:SCAR
- added U$23, U$25: (no value), shapes:LIGHTNING
- moved U$8 3.45 mm to (80.0, 50.8)
- moved R14 1.27 mm to (84.6, 54.6)
- moved LED4 1.27 mm to (89.4, 54.6)
- moved U$30 0.57 mm to (6.35, 77.7)
- moved U$31 0.57 mm to (6.35, 71.6)
- moved H1 0.25 mm to (59.4, 61.5)
- moved H2 0.25 mm to (34.5, 61.5)
- moved LED10 0.25 mm to (51.4, 74.3)
- moved LED11 0.25 mm to (42.5, 74.3)
- moved LED12 0.25 mm to (32.6, 74.3)
- moved LED13 0.25 mm to (22.7, 74.3)
- moved LED14 0.25 mm to (12.6, 74.3)
- moved LED7 0.25 mm to (80.9, 74.3)
- moved LED8 0.25 mm to (70.6, 74.3)
- moved LED9 0.25 mm to (61.1, 74.3)
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Routing:
- net IR_B_S: track 146.4 -> 154.1 mm, vias 0 -> 4
- net GND: track 828.4 -> 823.0 mm, vias 66 -> 76
- net +3V3: track 632.8 -> 634.9 mm
- net IR_A_S: track 202.2 -> 200.8 mm
- net N$31: track 5.72 -> 4.70 mm
- net N$16: track 219.8 -> 220.3 mm
Other:
- board size 94 x 82.8 mm -> 94.2 x 82.5 mm
